File: aux/aux.kicad_sch (KiCad schematic)
At the start: 25 parts

Commit message: Deployed 911a9c2 with MkDocs version: 1.5.3
Parts:
- added D?: LED_RGB, symbol Device:LED_RGB
Connections:
- net Earth: now also D?.1 (RK), D?.2 (GK), D?.3 (BK)
- net P3: now also D?.6 (RA)
- net P4: now also D?.5 (GA)
- net P5: now also D?.4 (BA)
Changed lines of the file:
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@@
   (junction (at 50.8 88.9) (diameter 0) (color 0 0 0 0)
   )
+  (junction (at 92.71 43.18) (diameter 0) (color 0 0 0 0)
+  )
   (junction (at 50.8 67.31) (diameter 0) (color 0 0 0 0)
   )
@@
     (stroke (width 0) (type default) (color 0 0 0 0))
   )
+  (wire (pts (xy 92.71 43.18) (xy 92.71 45.72))
+    (stroke (width 0) (type default) (color 0 0 0 0))
+  )
   (wire (pts (xy 38.1 99.06) (xy 40.64 99.06))
     (stroke (width 0) (type default) (color 0 0 0 0))
@@
     (stroke (width 0) (type default) (color 0 0 0 0))
   )
+  (wire (pts (xy 87.63 39.37) (xy 87.63 43.18))
+    (stroke (width 0) (type default) (color 0 0 0 0))
+  )
   (wire (pts (xy 48.26 111.76) (xy 50.8 111.76))
     (stroke (width 0) (type default) (color 0 0 0 0))
@@
     (stroke (width 0) (type default) (color 0 0 0 0))
   )
+  (wire (pts (xy 97.79 43.18) (xy 92.71 43.18))
+    (stroke (width 0) (type default) (color 0 0 0 0))
+  )
   (wire (pts (xy 48.26 80.01) (xy 50.8 80.01))
     (stroke (width 0) (type default) (color 0 0 0 0))
@@
     (stroke (width 0) (type default) (color 0 0 0 0))
   )
+  (wire (pts (xy 87.63 22.86) (xy 87.63 29.21))
+    (stroke (width 0) (type default) (color 0 0 0 0))
+  )
   (wire (pts (xy 50.8 67.31) (xy 50.8 73.66))
     (stroke (width 0) (type default) (color 0 0 0 0))
@@
     (stroke (width 0) (type default) (color 0 0 0 0))
   )
+  (wire (pts (xy 97.79 22.86) (xy 97.79 29.21))
+    (stroke (width 0) (type default) (color 0 0 0 0))
+  )
   (wire (pts (xy 50.8 80.01) (xy 50.8 86.36))
     (stroke (width 0) (type default) (color 0 0 0 0))
@@
     (stroke (width 0) (type default) (color 0 0 0 0))
   )
+  (wire (pts (xy 92.71 39.37) (xy 92.71 43.18))
+    (stroke (width 0) (type default) (color 0 0 0 0))
+  )
   (wire (pts (xy 50.8 60.96) (xy 50.8 67.31))
     (stroke (width 0) (type default) (color 0 0 0 0))
   )
+  (wire (pts (xy 92.71 22.86) (xy 92.71 29.21))
+    (stroke (width 0) (type default) (color 0 0 0 0))
+  )
   (wire (pts (xy 50.8 86.36) (xy 50.8 88.9))
     (stroke (width 0) (type default) (color 0 0 0 0))
@@
     (stroke (width 0) (type default) (color 0 0 0 0))
   )
+  (wire (pts (xy 97.79 39.37) (xy 97.79 43.18))
+    (stroke (width 0) (type default) (color 0 0 0 0))
+  )
   (wire (pts (xy 27.94 86.36) (xy 30.48 86.36))
     (stroke (width 0) (type default) (color 0 0 0 0))
   )
+  (wire (pts (xy 87.63 43.18) (xy 92.71 43.18))
+    (stroke (width 0) (type default) (color 0 0 0 0))
+  )
   (wire (pts (xy 58.42 35.56) (xy 58.42 38.1))
     (stroke (width 0) (type default) (color 0 0 0 0))
@@
   (wire (pts (xy 48.26 67.31) (xy 50.8 67.31))
     (stroke (width 0) (type default) (color 0 0 0 0))
+  )
+  (global_label "P3" (shape input) (at 87.63 22.86 90) (fields_autoplaced)
+    (effects (font (size 1.27 1.27)) (justify left))
+    (property "Referencias entre hojas" "${INTERSHEET_REFS}" (id 0) (at 87.5506 17.9674 90)
+      (effects (font (size 1.27 1.27)) (justify left) hide)
+    )
+  )
+  (global_label "P4" (shape input) (at 92.71 22.86 90) (fields_autoplaced)
+    (effects (font (size 1.27 1.27)) (justify left))
+    (property "Referencias entre hojas" "${INTERSHEET_REFS}" (id 0) (at 92.6306 17.9674 90)
+      (effects (font (size 1.27 1.27)) (justify left) hide)
+    )
   )
   (global_label "P4" (shape input) (at 27.94 86.36 180) (fields_autoplaced)
@@
     )
   )
+  (global_label "P5" (shape input) (at 97.79 22.86 90) (fields_autoplaced)
+    (effects (font (size 1.27 1.27)) (justify left))
+    (property "Referencias entre hojas" "${INTERSHEET_REFS}" (id 0) (at 97.7106 17.9674 90)
+      (effects (font (size 1.27 1.27)) (justify left) hide)
+    )
+  )
   (global_label "P6" (shape input) (at 27.94 99.06 180) (fields_autoplaced)
     (effects (font (size 1.27 1.27)) (justify right))
@@
     (pin "1")
     (pin "2")
+  )
+  (symbol (lib_id "power:Earth") (at 92.71 45.72 0) (unit 1)
+    (in_bom yes) (on_board yes) (fields_autoplaced)
+    (property "Reference" "#PWR?" (id 0) (at 92.71 52.07 0)
+      (effects (font (size 1.27 1.27)) hide)
+    )
+    (property "Value" "Earth" (id 1) (at 92.71 49.53 0)
+      (effects (font (size 1.27 1.27)) hide)
+    )
+    (property "Footprint" "" (id 2) (at 92.71 45.72 0)
+      (effects (font (size 1.27 1.27)) hide)
+    )
+    (property "Datasheet" "~" (id 3) (at 92.71 45.72 0)
+      (effects (font (size 1.27 1.27)) hide)
+    )
+    (pin "1")
   )
   (symbol (lib_id "Device:LED") (at 44.45 86.36 180) (unit 1)
@@
     (pin "2")
   )
+  (symbol (lib_id "Device:LED_RGB") (at 92.71 34.29 90) (unit 1)
+    (in_bom yes) (on_board yes) (fields_autoplaced)
+    (property "Reference" "D?" (id 0) (at 101.6 33.0199 90)
+      (effects (font (size 1.27 1.27)) (justify right) hide)
+    )
+    (property "Value" "LED_RGB" (id 1) (at 101.6 35.5599 90)
+      (effects (font (size 1.27 1.27)) (justify right) hide)
+    )
+    (property "Footprint" "" (id 2) (at 93.98 34.29 0)
+      (effects (font (size 1.27 1.27)) hide)
+    )
+    (property "Datasheet" "~" (id 3) (at 93.98 34.29 0)
+      (effects (font (size 1.27 1.27)) hide)
+    )
+    (pin "1")
+    (pin "2")
+    (pin "3")
+    (pin "4")
+    (pin "5")
+    (pin "6")
+  )
   (symbol (lib_id "Device:LED") (at 44.45 92.71 180) (unit 1)
     (in_bom yes) (on_board yes)
@@
   )
   (symbol_instances
+    (path "/04ef2036-83eb-41ea-bdaf-69afb04e0771"
+      (reference "#PWR?") (unit 1) (value "Earth") (footprint "")
+    )
     (path "/1cf4ff77-aa55-4a27-8859-0548ad057b70"
       (reference "#PWR?") (unit 1) (value "Earth") (footprint "")
@@
       (reference "D?") (unit 1) (value "segmento") (footprint "")
     )
+    (path "/ac85b0e1-331b-4079-9e85-e331d3d2bfe1"
+      (reference "D?") (unit 1) (value "LED_RGB") (footprint "")
+    )
     (path "/b07e92d3-4b63-4768-98b2-27c9824179d5"

Commit message: Deployed 5b4c9c1c with MkDocs version: 1.5.3
Parts:
- added BZ? (x2): Buzzer, symbol Device:Buzzer
- added D?: Amarillo, symbol Device:LED
- added D?: Verde, symbol Device:LED
- added D?: Rojo, symbol Device:LED
- added Q? (x2): Q_NPN_BCE, symbol Device:Q_NPN_BCE
- added R? (x3): 220 (op), symbol Device:R
- added R? (x3): 10K, symbol Device:R
- added R? (x2): 1k, symbol Device:R
- added SW? (x2): SW_Push, symbol Switch:SW_Push
Connections:
- net +3.3V: now also BZ?.1 (-), BZ?.1 (-), R?.1, SW?.2
- net Earth: now also D?.1 (K), D?.1 (K), D?.1 (K), Q?.3 (E), Q?.3 (E), R?.2, SW?.1
- net P1: now also R?.1, R?.1
- net P2: now also R?.1, R?.2, SW?.1
- net P3: now also R?.1
- net P4: now also R?.1
- net P5: now also R?.1
- new net: R?.1, R?.2, SW?.2
- new net: D?.2 (A), R?.2 (x3)
- new net: BZ?.2 (+), Q?.2 (C) (x2)
- new net: Q?.1 (B), R?.2 (x2)
